File: probe_sys1.kicad_pcb (KiCad board)
At the start: 2 copper layers, 90 x 90 mm, 41 parts, among them J1 Screw_Terminal_01x02

Commit message: RPI, RN, ESP.
Parts:
- removed D1, D2: LED, LED_SMD:LED_0603_1608Metric_Pad1.05x0.95mm_HandSolder
- removed J1: Screw_Terminal_01x02, PEP_library:TerminalBlock_Phoenix_MKDS-1,5-2-5.08_1x02_P5.08mm_Horizontal
- removed JP1, JP2, JP3, JP4, JP5, JP6, JP7, JP8: Jumper, Connector_PinHeader_2.54mm:PinHeader_1x02_P2.54mm_Vertical
- removed R1, R6: 300, PEP_library:R_smd
- removed R2, R3, R5, R8: 4.7k, PEP_library:R_smd
- removed R4, R7: 1k, PEP_library:R_smd
- removed REF**: ele_petnica_logo, PEP_library:ele_petnica_logo
- removed REF** (x8): JP_silk_symbol, PEP_library:JP_silk_symbol
- removed REF** (x8): R_silk_symbol, PEP_library:R_silk_symbol
- added MODULE1: RN2483-I_RM095, probe_sys1:RN2483-I_RM095, F.Cu at (143.4, 109.8)
- added U1: ESP32-WROOM-32UE, RF_Module:ESP32-WROOM-32UE, F.Cu at (164.2, 105.9)
- added U2: RASPBERRY_PI_ZERO_2_W, probe_sys1:MODULE_RASPBERRY_PI_ZERO_2_W, F.Cu at (145.0, 68.0)
Routing:
- net 0: track 73.7 -> 0.00 mm
- net 9V: track 64.0 -> 0.00 mm
- net Net-(D2-A): track 30.2 -> 0.00 mm
- net Net-(D1-A): track 30.1 -> 0.00 mm
- net Net-(JP1-B): track 22.6 -> 0.00 mm
- net Net-(JP3-B): track 22.5 -> 0.00 mm
- net Net-(JP2-B): track 22.2 -> 0.00 mm
- net Net-(JP8-B): track 8.95 -> 0.00 mm
- net Net-(JP7-B): track 8.69 -> 0.00 mm
- net Net-(JP6-B): track 8.69 -> 0.00 mm
- net Net-(JP5-B): track 8.45 -> 0.00 mm

Commit message: SIM, wroom.
Parts:
- added U3: SIM808, probe_sys1:SIM808, F.Cu at (117.0, 110.2)
- U1: footprint RF_Module:ESP32-WROOM-32UE -> probe_sys1:ESP32-WROOM-32UE
- moved U1 2.07 mm to (166.0, 107.0)
